Commit message: fix scales

File: ANDPS/panda_images/urdfs/angle_box/angle_box.urdf (robot description, URDF)
Before this commit: robot angle_box, 1 links, 0 joints
Links:
- link base_link: geometry collision mesh filename=angle_box.dae scale=0.1 1 1; visual mesh filename=angle_box.dae scale=0.1 1 1
