Commit message: some updates

File: ANDPS/rl_pour/urdfs/bowl/bowl.urdf (robot description, URDF)
Before this commit: robot bowl, 1 links, 0 joints
Links:
- link base_link: geometry collision mesh filename=bowl.dae scale=0.05 0.05 0.05; visual mesh filename=bowl.dae scale=0.05 0.05 0.05

File: ANDPS/rl_pour/urdfs/cheerio/cheerio.urdf (robot description, URDF)
Before this commit: robot cereal, 1 links, 0 joints
Links:
- link base_link: geometry collision mesh filename=cheerio.dae scale=2 2 2; visual mesh filename=cheerio.dae scale=2 2 2
