Commit message: simpler env

File: ANDPS/rl_pour/urdfs/franka/franka.urdf (robot description, URDF)
Before this commit: robot panda, 14 links, 13 joints
Links:
- link cereal_box: geometry collision mesh filename=package://franka_description/meshes/collision/cereal.stl scale=0.8 0.8 0.8; visual mesh filename=package://franka_description/meshes/visual/cereal.dae scale=0.8 0.8 0.8

File: ANDPS/rl_pour/urdfs/table/table.urdf (robot description, URDF)
Before this commit: robot table, 1 links, 0 joints
Links:
- link base_link: geometry collision mesh filename=table.stl scale=1 1 1; visual mesh filename=table_3.dae scale=1 1 1

Commit message: boxes for collisions

File: ANDPS/rl_pour/urdfs/franka/franka.urdf (robot description, URDF)
Before this commit: robot panda, 14 links, 13 joints
Links:
- link cereal_box: geometry collision box size=0.04 0.3 0.3; visual mesh filename=package://franka_description/meshes/visual/cereal.dae scale=0.8 0.8 0.8

Commit message: more changes

File: ANDPS/rl_pour/urdfs/franka/franka.urdf (robot description, URDF)
Before this commit: robot panda, 14 links, 13 joints
Links:
- removed link panda_leftfinger
- removed link panda_rightfinger
- link cereal_box: geometry collision box size=0.02 0.07 0.07; collision box size=0.09 0.02 0.07
Joints:
- removed joint panda_finger_joint1
- removed joint panda_finger_joint2
- joint cereal_joint: parent panda_leftfinger -> panda_ee

Commit message: more changes

File: ANDPS/rl_pour/urdfs/franka/franka.urdf (robot description, URDF)
Before this commit: robot panda, 12 links, 11 joints
Links:
- link cereal_box: geometry collision box size=0.02 0.07 0.07; collision box size=0.12 0.02 0.07
